Commit message: more stuff

File: crew_systems/workspace_analysis/sawyer/urdf/sawyer.urdf (robot description, URDF)
Before this commit: robot sawyer, 21 links, 20 joints
Links:
- removed link head
- removed link head_camera
- removed link screen
Joints:
- removed joint display_joint
- removed joint head_camera
- removed joint head_pan
