Commit message: made some changes, added some images

File: crew_systems/workspace_analysis/rover_crane/urdf/rover_crane.urdf (robot description, URDF)
Before this commit: robot rover_crane, 5 links, 4 joints
Links:
- removed link base_link
- added link rover_base_link; collision box size=2.6 1.5 0.5; collision box size=6 6 0.01
Joints:
- removed joint joint1
- removed joint joint2
- removed joint joint3
- added joint joint0_1: type revolute, parent rover_base_link, child crane_yaw, origin xyz=1.1 0 0.5 rpy=0 0 0, axis 0 0 1, limit lower=-0.523599 upper=0.523599 effort=0 velocity=0
- added joint joint0_2: type revolute, parent crane_yaw, child crane_link1, origin xyz=0 0 0.3 rpy=0 1.5708 0, axis 0 1 0, limit lower=0.0 upper=1.5708 effort=0 velocity=0
- added joint joint0_3: type prismatic, parent crane_link1, child crane_link2, origin xyz=-3.396 0 0 rpy=0 0 0, axis -1 0 0, limit lower=0.0 upper=2.264 effort=0 velocity=0

File: crew_systems/workspace_analysis/rover_crane/urdf/rover_crane_nbv.urdf (robot description, URDF)
Before this commit: robot rover_crane_nbv, 12 links, 11 joints
Links:
- link rover_base_link: geometry collision box size=2.6 1.5 0.5; collision box size=6 6 0.01
Joints:
- joint joint0_1: origin xyz=1.0 0 0.5 rpy=0 0 0 -> xyz=1.1 0 0.5 rpy=0 0 0

File: crew_systems/workspace_analysis/rover_crane/urdf/rover_crane_sawyer.urdf (robot description, URDF)
Before this commit: robot rover_crane_sawyer, 23 links, 22 joints
Links:
- link rover_base_link: geometry collision box size=2.6 1.5 0.5; collision box size=6 6 0.01
Joints:
- joint joint0_1: origin xyz=1.0 0 0.5 rpy=0 0 0 -> xyz=1.1 0 0.5 rpy=0 0 0
- joint tip_joint: origin xyz=0 0 -0.1 rpy=0 -1.261657 0 -> xyz=0 0 -0.1 rpy=0 -1.26165662836 0
