Commit message: more stuff and /or things

File: crew_systems/workspace_analysis/rover_crane/urdf/rover_crane/rover_crane_old1.urdf (robot description, URDF)
Before this commit: robot rover_crane, 5 links, 4 joints
Links:
- link rover_base_link: geometry collision box size=2.4 1.5 0.5; visual box size=2.4 1.5 0.5
Joints:
- joint joint0_1: origin xyz=1.1 0 0.5 rpy=0 0 0 -> xyz=1 0 0.5 rpy=0 0 0
