Commit message: balling, but at what cost?

File: crew_systems/workspace_analysis/rover_crane/urdf/crane/crane_old2.urdf (robot description, URDF)
Before this commit: robot crane, 6 links, 5 joints
Links:
- added link tip; collision box size=0.2 0.2 1.0; visual box size=0.2 0.2 1.0
Joints:
- added joint tip_joint: type fixed, parent crane_link4, child tip, origin xyz=0 0 0 rpy=0 -0.371755130675 0
