Commit message: balling

File: crew_systems/workspace_analysis/nbv/urdf/nbv_for_density_xz.urdf (robot description, URDF)
Before this commit: robot nbv, 8 links, 7 joints
Joints:
- removed joint wold_rotate
- added joint world_rotate: type fixed, parent ground, child base_link, origin xyz=0 0 0 rpy=-1.5708 0 0
