Commit message: pain?

File: crew_systems/workspace_analysis/dymaflight/urdf/dymaflight.urdf (robot description, URDF)
Before this commit: robot dymaflight, 5 links, 4 joints
Links:
- added link tool_roll; collision mesh filename=package://nbv/urdf/meshes/tool_roll.stl scale=0.001 0.001 0.001; visual mesh filename=package://nbv/urdf/meshes/tool_roll.stl scale=0.001 0.001 0.001
- added link wrst_ptch; collision mesh filename=package://nbv/urdf/meshes/wrst_ptch.stl scale=0.001 0.001 0.001; visual mesh filename=package://nbv/urdf/meshes/wrst_ptch.stl scale=0.001 0.001 0.001
- added link wrst_roll; collision mesh filename=package://nbv/urdf/meshes/wrst_roll.stl scale=0.001 0.001 0.001; visual mesh filename=package://nbv/urdf/meshes/wrst_roll.stl scale=0.001 0.001 0.001
Joints:
- added joint joint5: type revolute, parent elbw_ptch, child wrst_roll, origin xyz=0.041402 0.37084 0 rpy=-1.5708 0 0, axis 0 0 1, limit lower=-3.14159 upper=3.14159 effort=300 velocity=0.25
- added joint joint6: type revolute, parent wrst_roll, child wrst_ptch, origin xyz=0.033274 -0.007366 0 rpy=-1.5708 0 3.14159, axis 0 0 1, limit lower=-3.14159 upper=3.14159 effort=300 velocity=0.25
- added joint joint7: type revolute, parent wrst_ptch, child tool_roll, origin xyz=0.033274 0 0 rpy=1.5708 0 0, axis 0 0 1, limit lower=-3.14159 upper=3.14159 effort=300 velocity=0.25
- joint joint2: origin xyz=0 0 0 rpy=0 -1.5708 1.5708 -> xyz=0 0 0 rpy=-1.5708 0 3.14159 
- joint joint4: origin xyz=0.041402 0 0 rpy=-1.5708 -1.5708 0 -> xyz=0.041402 0 0 rpy=-1.5708 -3.14159 0

File: crew_systems/workspace_analysis/rover_crane/urdf/rover_crane/rover_crane_old2.urdf (robot description, URDF)
Before this commit: robot rover_crane, 8 links, 7 joints
Joints:
- joint tip_joint: parent cclrane_link4 -> crane_link4

Commit message: balling

File: crew_systems/workspace_analysis/dymaflight/urdf/dymaflight.urdf (robot description, URDF)
Before this commit: robot dymaflight, 8 links, 7 joints
Links:
- link elbw_ptch: geometry collision mesh filename=package://dymaflight/urdf/meshes/elbw_ptch.stl scale=0.001 0.001 0.001; visual mesh filename=package://dymaflight/urdf/meshes/elbw_ptch.stl scale=0.001 0.001 0.001
- link shld_ptch: geometry collision mesh filename=package://dymaflight/urdf/meshes/shld_ptch.stl scale=0.001 0.001 0.001; visual mesh filename=package://dymaflight/urdf/meshes/shld_ptch.stl scale=0.001 0.001 0.001
- link shld_roll: geometry collision mesh filename=package://dymaflight/urdf/meshes/shld_roll.stl scale=0.001 0.001 0.001; visual mesh filename=package://dymaflight/urdf/meshes/shld_roll.stl scale=0.001 0.001 0.001
- link shld_yaw: geometry collision mesh filename=package://dymaflight/urdf/meshes/shld_yaw.stl scale=0.001 0.001 0.001; visual mesh filename=package://dymaflight/urdf/meshes/shld_yaw.stl scale=0.001 0.001 0.001
- link tool_roll: geometry collision mesh filename=package://dymaflight/urdf/meshes/tool_roll.stl scale=0.001 0.001 0.001; visual mesh filename=package://dymaflight/urdf/meshes/tool_roll.stl scale=0.001 0.001 0.001
- link wrst_ptch: geometry collision mesh filename=package://dymaflight/urdf/meshes/wrst_ptch.stl scale=0.001 0.001 0.001; visual mesh filename=package://dymaflight/urdf/meshes/wrst_ptch.stl scale=0.001 0.001 0.001
- link wrst_roll: geometry collision mesh filename=package://dymaflight/urdf/meshes/wrst_roll.stl scale=0.001 0.001 0.001; visual mesh filename=package://dymaflight/urdf/meshes/wrst_roll.stl scale=0.001 0.001 0.001
